File: hardware/esp32-m2-breadboard.sch (KiCad schematic (older format))
At the start: 4 parts, among them J1 2199230-4, J2 Conn_01x16_Female, J3 Conn_01x16_Female

Commit message: Pins assigned
Parts:
- J2, J3: value Conn_01x16_Female -> Conn_01x15_Female; footprint Connector_PinHeader_2.54mm:PinHeader_1x16_P2.54mm_Vertical -> Connector_PinHeader_2.54mm:PinHeader_1x15_P2.54mm_Vertical; symbol Connector:Conn_01x16_Female -> Connector:Conn_01x15_Female
Connections:
- net labels added: +5V, DTR, GND, GPIO15, GPIO16, GPIO18, GPIO19, GPIO2, GPIO21, GPIO22, GPIO23, GPIO25-DAC1, GPIO26-DAC2, GPIO27, GPIO32, GPIO33, GPIO4, GPIO5, RESET, RTS, RX, TX
- wire segments 0 -> 86
- no-connect marks 0 -> 34
Other:
- moved on the sheet: MP1
