File: hardware/esp32-m2-breadboard.kicad_pcb (KiCad board)
At the start: 2 copper layers, 57.2 x 22.9 mm, 4 parts, among them J1 2199230-4, J2 Conn_01x15_Female, J3 Conn_01x15_Female

Commit message: Set version of previous commit to board
Other:
- board text added: "François Gervais 19 jan 2021 v1.0-1-g1b0212e"
- board text removed: "François Gervais 19 jan 2021 Rev 1.0"
